File: eagle/sputnik_prototype_SysController.sch (EAGLE design)
At the start: 69 parts, among them SW1 TPS25944LRVCRWQFN-20-3X4, U1 MEGA128-A, X1 CRYSTAL-ABRACON-ABM3-SMD

Commit message: A few more changes
Parts:
- removed TP4, TP5: TPSPAD1-13, testpad:TPSPAD1-13
- added C10: Value, rcl_custom:C-EU0402-B-NOSILK
- added TP28, TP29: TPSPAD1-13, testpad:TPSPAD1-13
- Q1: device transistor-power:N-MOSFET-SO8S -> adafruit:MOSFET-NREFLOW
Connections:
- removed net N$7: SW1.!FLT, TP5.PP
- new net N$25: SW1.PGOOD, TP29.PP
- new net N$28: SW1.PGHT, TP28.PP
- new net N$29: SW1.!FLT
- new net N$31: C10.1, SW1.DV/DT
- net GND: now also C10.2; no longer SW1.DV/DT, SW1.PGHT, SW1.PGOOD
- net N$27: no longer TP4.PP
Other:
- note added: "Set UVLO to 3.0V"
- note added: "Todo: Find a new MOSFET: PMPB29XNE IRLHS6242TR2PBF Find a 16:1 multiplexer: MAX14661 74HC4067; 74HCT4067 Determine ILIM for each switch"
- note added: "V+"
- note removed: "Todo: Find a new MOSFET: PMPB29XNE I RLHS6242TR2PBF Find a 16:1 multiplexer: MAX14661 74HC4067; 74HCT4067 Determine ILIM for each switch"
- note removed: "Vin"
Changed lines of the file:
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@@
 <part name="RUVLO" library="rcl_custom" deviceset="R-US_" device="0603-B-NOSILK" value="Value"/>
 <part name="R6" library="rcl_custom" deviceset="R-US_" device="0603-B-NOSILK" value="Value"/>
-<part name="Q1" library="transistor-power" deviceset="N-MOSFET-SO8" device="S"/>
 <part name="RILIM" library="rcl_custom" deviceset="R-US_" device="0603-B-NOSILK" value="Value"/>
 <part name="GND4" library="psas_c3_team05" deviceset="GND" device=""/>
 <part name="RIMON" library="rcl_custom" deviceset="R-US_" device="0603-B-NOSILK" value="Value"/>
-<part name="TP4" library="testpad" deviceset="TPS" device="PAD1-13"/>
 <part name="C9" library="rcl_custom" deviceset="C-EU" device="0402-B-NOSILK" value="1uF"/>
 <part name="GND2" library="psas_c3_team05" deviceset="GND" device=""/>
-<part name="TP5" library="testpad" deviceset="TPS" device="PAD1-13"/>
+<part name="TP28" library="testpad" deviceset="TPS" device="PAD1-13"/>
+<part name="TP29" library="testpad" deviceset="TPS" device="PAD1-13"/>
+<part name="C10" library="rcl_custom" deviceset="C-EU" device="0402-B-NOSILK" value="Value"/>
+<part name="Q1" library="adafruit" deviceset="MOSFET-N" device="REFLOW"/>
 </parts>
 <sheets>
@@
 Find a new MOSFET:
      PMPB29XNE
-I    RLHS6242TR2PBF
+     IRLHS6242TR2PBF
 Find a 16:1 multiplexer:
      MAX14661
@@
 <text x="327.66" y="317.5" size="1.778" layer="97">Vout</text>
 <text x="327.66" y="314.96" size="1.778" layer="97">!FLT</text>
-<text x="231.14" y="317.5" size="1.778" layer="97">Vin</text>
+<text x="231.14" y="317.5" size="1.778" layer="97">V+</text>
 <text x="228.6" y="297.18" size="1.778" layer="97">Enable</text>
 <text x="327.66" y="307.34" size="1.778" layer="97">IMON</text>
@@
 <wire x1="228.6" y1="281.94" x2="228.6" y2="350.52" width="0.1524" layer="97" style="longdash"/>
 <wire x1="228.6" y1="350.52" x2="335.28" y2="350.52" width="0.1524" layer="97" style="longdash"/>
+<text x="238.76" y="320.04" size="1.778" layer="97">Set UVLO to 3.0V</text>
 </plain>
 <instances>
@@
 </instance>
 <instance part="R6" gate="R" x="251.46" y="297.18" rot="R270"/>
-<instance part="Q1" gate="G$1" x="238.76" y="299.72"/>
 <instance part="RILIM" gate="R" x="297.18" y="297.18" smashed="yes" rot="R270">
 <attribute name="NAME" x="298.6786" y="300.99" size="1.778" layer="95" rot="R270"/>
@@
 <attribute name="VALUE" x="301.498" y="300.99" size="1.778" layer="96" rot="R270"/>
 </instance>
-<instance part="TP4" gate="G$1" x="299.72" y="309.88"/>
 <instance part="C9" gate="CE" x="256.54" y="314.96"/>
 <instance part="GND2" gate="1" x="256.54" y="307.34"/>
-<instance part="TP5" gate="G$1" x="299.72" y="317.5"/>
+<instance part="TP28" gate="G$1" x="299.72" y="312.42"/>
+<instance part="TP29" gate="G$1" x="299.72" y="314.96"/>
+<instance part="C10" gate="CE" x="261.62" y="299.72" smashed="yes">
+<attribute name="NAME" x="263.144" y="300.101" size="1.778" layer="95"/>
+<attribute name="VALUE" x="263.144" y="295.021" size="1.778" layer="96"/>
+</instance>
+<instance part="Q1" gate="G$1" x="238.76" y="299.72"/>
 </instances>
 <busses>
@@
 <pinref part="SW1" gate="G$1" pin="GND"/>
 <wire x1="266.7" y1="304.8" x2="264.16" y2="304.8" width="0.1524" layer="91"/>
-<wire x1="264.16" y1="304.8" x2="264.16" y2="307.34" width="0.1524" layer="91"/>
-<pinref part="SW1" gate="G$1" pin="DV/DT"/>
-<wire x1="266.7" y1="307.34" x2="264.16" y2="307.34" width="0.1524" layer="91"/>
 <pinref part="SW1" gate="G$1" pin="DMODE"/>
 <wire x1="266.7" y1="309.88" x2="264.16" y2="309.88" width="0.1524" layer="91"/>
@@
 <pinref part="SW1" gate="G$1" pin="OVP"/>
 <wire x1="266.7" y1="312.42" x2="264.16" y2="312.42" width="0.1524" layer="91"/>
-<wire x1="264.16" y1="309.88" x2="264.16" y2="307.34" width="0.1524" layer="91"/>
+<wire x1="264.16" y1="309.88" x2="264.16" y2="304.8" width="0.1524" layer="91"/>
 <wire x1="264.16" y1="304.8" x2="264.16" y2="292.1" width="0.1524" layer="91"/>
 <pinref part="GND1" gate="1" pin="GND"/>
 <pinref part="R6" gate="R" pin="2"/>
-<wire x1="251.46" y1="292.1" x2="264.16" y2="292.1" width="0.1524" layer="91"/>
-<pinref part="Q1" gate="G$1" pin="S"/>
+<wire x1="251.46" y1="292.1" x2="261.62" y2="292.1" width="0.1524" layer="91"/>
+<wire x1="261.62" y1="292.1" x2="264.16" y2="292.1" width="0.1524" layer="91"/>
 <wire x1="241.3" y1="294.64" x2="241.3" y2="292.1" width="0.1524" layer="91"/>
 <wire x1="241.3" y1="292.1" x2="251.46" y2="292.1" width="0.1524" layer="91"/>
 <junction x="251.46" y="292.1"/>
+<junction x="264.16" y="304.8"/>
+<junction x="264.16" y="309.88"/>
+<junction x="264.16" y="292.1"/>
+<pinref part="C10" gate="CE" pin="2"/>
+<wire x1="261.62" y1="294.64" x2="261.62" y2="292.1" width="0.1524" layer="91"/>
+<junction x="261.62" y="292.1"/>
+<pinref part="Q1" gate="G$1" pin="S"/>
 </segment>
 <segment>
@@
 <wire x1="297.18" y1="292.1" x2="297.18" y2="289.56" width="0.1524" layer="91"/>
 <pinref part="GND4" gate="1" pin="GND"/>
-<pinref part="SW1" gate="G$1" pin="PGOOD"/>
-<wire x1="297.18" y1="312.42" x2="299.72" y2="312.42" width="0.1524" layer="91"/>
-<wire x1="299.72" y1="312.42" x2="312.42" y2="312.42" width="0.1524" layer="91"/>
-<wire x1="312.42" y1="312.42" x2="312.42" y2="289.56" width="0.1524" layer="91"/>
-<wire x1="312.42" y1="289.56" x2="304.8" y2="289.56" width="0.1524" layer="91"/>
 <pinref part="RIMON" gate="R" pin="2"/>
+<wire x1="304.8" y1="292.1" x2="304.8" y2="289.56" width="0.1524" layer="91"/>
 <wire x1="304.8" y1="289.56" x2="297.18" y2="289.56" width="0.1524" layer="91"/>
-<wire x1="304.8" y1="292.1" x2="304.8" y2="289.56" width="0.1524" layer="91"/>
-<junction x="304.8" y="289.56"/>
-<pinref part="SW1" gate="G$1" pin="PGHT"/>
-<wire x1="297.18" y1="309.88" x2="299.72" y2="309.88" width="0.1524" layer="91"/>
-<wire x1="299.72" y1="309.88" x2="299.72" y2="312.42" width="0.1524" layer="91"/>
-<junction x="299.72" y="312.42"/>
+<junction x="297.18" y="289.56"/>
 </segment>
 <segment>
@@
 <net name="N$7" class="0">
 <segment>
-<pinref part="SW1" gate="G$1" pin="!FLT"/>
-<wire x1="297.18" y1="314.96" x2="299.72" y2="314.96" width="0.1524" layer="91"/>
-<pinref part="TP5" gate="G$1" pin="PP"/>
 <wire x1="299.72" y1="314.96" x2="332.74" y2="314.96" width="0.1524" layer="91"/>
-<junction x="299.72" y="314.96"/>
 </segment>
 </net>
@@
 <segment>
 <pinref part="SW1" gate="G$1" pin="EN/UVLO"/>
-<wire x1="266.7" y1="314.96" x2="261.62" y2="314.96" width="0.1524" layer="91"/>
-<wire x1="261.62" y1="314.96" x2="261.62" y2="304.8" width="0.1524" layer="91"/>
+<wire x1="266.7" y1="314.96" x2="259.08" y2="314.96" width="0.1524" layer="91"/>
+<wire x1="259.08" y1="314.96" x2="259.08" y2="304.8" width="0.1524" layer="91"/>
 <pinref part="RUVLO" gate="R" pin="2"/>
 <wire x1="251.46" y1="307.34" x2="251.46" y2="304.8" width="0.1524" layer="91"/>
 <pinref part="R6" gate="R" pin="1"/>
-<pinref part="Q1" gate="G$1" pin="D"/>
 <wire x1="251.46" y1="304.8" x2="251.46" y2="302.26" width="0.1524" layer="91"/>
 <wire x1="241.3" y1="304.8" x2="251.46" y2="304.8" width="0.1524" layer="91"/>
-<wire x1="261.62" y1="304.8" x2="251.46" y2="304.8" width="0.1524" layer="91"/>
+<wire x1="259.08" y1="304.8" x2="251.46" y2="304.8" width="0.1524" layer="91"/>
 <junction x="251.46" y="304.8"/>
+<pinref part="Q1" gate="G$1" pin="D"/>
 </segment>
 </net>
 <net name="N$26" class="0">
 <segment>
+<wire x1="236.22" y1="297.18" x2="231.14" y2="297.18" width="0.1524" layer="91"/>
 <pinref part="Q1" gate="G$1" pin="G"/>
-<wire x1="236.22" y1="297.18" x2="231.14" y2="297.18" width="0.1524" layer="91"/>
 </segment>
 </net>
@@
 <wire x1="304.8" y1="307.34" x2="304.8" y2="302.26" width="0.1524" layer="91"/>
 <wire x1="304.8" y1="307.34" x2="299.72" y2="307.34" width="0.1524" layer="91"/>
-<pinref part="TP4" gate="G$1" pin="PP"/>
-<wire x1="299.72" y1="307.34" x2="332.74" y2="307.34" width="0.1524" layer="91"/>
+<wire x1="304.8" y1="307.34" x2="332.74" y2="307.34" width="0.1524" layer="91"/>
 <junction x="304.8" y="307.34"/>
 </segment>
 </net>
+<net name="N$25" class="0">
+<segment>
+<pinref part="SW1" gate="G$1" pin="PGOOD"/>
+<wire x1="297.18" y1="312.42" x2="299.72" y2="312.42" width="0.1524" layer="91"/>
+<pinref part="TP29" gate="G$1" pin="PP"/>
+</segment>
+</net>
+<net name="N$28" class="0">
+<segment>
+<pinref part="SW1" gate="G$1" pin="PGHT"/>
+<wire x1="297.18" y1="309.88" x2="299.72" y2="309.88" width="0.1524" layer="91"/>
+<pinref part="TP28" gate="G$1" pin="PP"/>
+</segment>
+</net>
+<net name="N$29" class="0">
+<segment>
+<pinref part="SW1" gate="G$1" pin="!FLT"/>
+<wire x1="297.18" y1="314.96" x2="304.8" y2="314.96" width="0.1524" layer="91"/>
+</segment>
+</net>
+<net name="N$31" class="0">
+<segment>
+<pinref part="SW1" gate="G$1" pin="DV/DT"/>
+<wire x1="266.7" y1="307.34" x2="261.62" y2="307.34" width="0.1524" layer="91"/>
+<wire x1="261.62" y1="307.34" x2="261.62" y2="302.26" width="0.1524" layer="91"/>
+<pinref part="C10" gate="CE" pin="1"/>
+</segment>
+</net>

Commit message: latest changes
Parts:
- Q1: value (none) -> IRLML6344TRPBF; device adafruit:MOSFET-NREFLOW -> adafruit:IRLML6344TRPBF
Other:
- note added: "Todo: Find a 16:1 multiplexer: MAX14661 74HC4067; 74HCT4067 Determine ILIM for each switch"
- note removed: "Todo: Find a new MOSFET: PMPB29XNE IRLHS6242TR2PBF Find a 16:1 multiplexer: MAX14661 74HC4067; 74HCT4067 Determine ILIM for each switch"
Changed lines of the file:
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@@
 <part name="TP29" library="testpad" deviceset="TPS" device="PAD1-13"/>
 <part name="C10" library="rcl_custom" deviceset="C-EU" device="0402-B-NOSILK" value="Value"/>
-<part name="Q1" library="adafruit" deviceset="MOSFET-N" device="REFLOW"/>
+<part name="Q1" library="adafruit" deviceset="IRLML6344TRPBF" device=""/>
 </parts>
 <sheets>
@@
 9.ADS-Starfinder/Sunsensor</text>
 <text x="231.14" y="327.66" size="1.778" layer="97">Todo:
-Find a new MOSFET:
-     PMPB29XNE
-     IRLHS6242TR2PBF
 Find a 16:1 multiplexer:
      MAX14661
@@
 <text x="327.66" y="314.96" size="1.778" layer="97">!FLT</text>
 <text x="231.14" y="317.5" size="1.778" layer="97">V+</text>
-<text x="228.6" y="297.18" size="1.778" layer="97">Enable</text>
+<text x="231.14" y="294.64" size="1.778" layer="97">Enable</text>
 <text x="327.66" y="307.34" size="1.778" layer="97">IMON</text>
 <wire x1="335.28" y1="350.52" x2="335.28" y2="281.94" width="0.1524" layer="97" style="longdash"/>
@@
 </instance>
 <instance part="SW1" gate="G$1" x="281.94" y="309.88"/>
-<instance part="GND1" gate="1" x="264.16" y="289.56"/>
+<instance part="GND1" gate="1" x="264.16" y="287.02"/>
 <instance part="RUVLO" gate="R" x="251.46" y="312.42" smashed="yes" rot="R270">
 <attribute name="NAME" x="252.9586" y="316.23" size="1.778" layer="95" rot="R270"/>
@@
 <attribute name="VALUE" x="263.144" y="295.021" size="1.778" layer="96"/>
 </instance>
-<instance part="Q1" gate="G$1" x="238.76" y="299.72"/>
+<instance part="Q1" gate="G$1" x="241.3" y="297.18" smashed="yes">
+<attribute name="NAME" x="238.76" y="300.355" size="1.27" layer="95"/>
+<attribute name="VALUE" x="246.38" y="290.83" size="1.27" layer="96" rot="R90"/>
+</instance>
 </instances>
 <busses>
@@
 <wire x1="266.7" y1="312.42" x2="264.16" y2="312.42" width="0.1524" layer="91"/>
 <wire x1="264.16" y1="309.88" x2="264.16" y2="304.8" width="0.1524" layer="91"/>
-<wire x1="264.16" y1="304.8" x2="264.16" y2="292.1" width="0.1524" layer="91"/>
+<wire x1="264.16" y1="304.8" x2="264.16" y2="289.56" width="0.1524" layer="91"/>
 <pinref part="GND1" gate="1" pin="GND"/>
-<pinref part="R6" gate="R" pin="2"/>
-<wire x1="251.46" y1="292.1" x2="261.62" y2="292.1" width="0.1524" layer="91"/>
-<wire x1="261.62" y1="292.1" x2="264.16" y2="292.1" width="0.1524" layer="91"/>
-<wire x1="241.3" y1="294.64" x2="241.3" y2="292.1" width="0.1524" layer="91"/>
-<wire x1="241.3" y1="292.1" x2="251.46" y2="292.1" width="0.1524" layer="91"/>
-<junction x="251.46" y="292.1"/>
+<wire x1="261.62" y1="289.56" x2="264.16" y2="289.56" width="0.1524" layer="91"/>
 <junction x="264.16" y="304.8"/>
 <junction x="264.16" y="309.88"/>
-<junction x="264.16" y="292.1"/>
+<junction x="264.16" y="289.56"/>
 <pinref part="C10" gate="CE" pin="2"/>
-<wire x1="261.62" y1="294.64" x2="261.62" y2="292.1" width="0.1524" layer="91"/>
-<junction x="261.62" y="292.1"/>
+<wire x1="261.62" y1="294.64" x2="261.62" y2="289.56" width="0.1524" layer="91"/>
+<wire x1="243.84" y1="292.1" x2="243.84" y2="289.56" width="0.1524" layer="91"/>
+<wire x1="243.84" y1="289.56" x2="251.46" y2="289.56" width="0.1524" layer="91"/>
+<wire x1="261.62" y1="289.56" x2="251.46" y2="289.56" width="0.1524" layer="91"/>
+<pinref part="R6" gate="R" pin="2"/>
+<wire x1="251.46" y1="289.56" x2="251.46" y2="292.1" width="0.1524" layer="91"/>
+<junction x="251.46" y="289.56"/>
+<junction x="261.62" y="289.56"/>
 <pinref part="Q1" gate="G$1" pin="S"/>
 </segment>
@@
 <pinref part="R6" gate="R" pin="1"/>
 <wire x1="251.46" y1="304.8" x2="251.46" y2="302.26" width="0.1524" layer="91"/>
-<wire x1="241.3" y1="304.8" x2="251.46" y2="304.8" width="0.1524" layer="91"/>
 <wire x1="259.08" y1="304.8" x2="251.46" y2="304.8" width="0.1524" layer="91"/>
 <junction x="251.46" y="304.8"/>
+<wire x1="243.84" y1="302.26" x2="243.84" y2="304.8" width="0.1524" layer="91"/>
+<wire x1="243.84" y1="304.8" x2="251.46" y2="304.8" width="0.1524" layer="91"/>
 <pinref part="Q1" gate="G$1" pin="D"/>
 </segment>
@@
 <net name="N$26" class="0">
 <segment>
-<wire x1="236.22" y1="297.18" x2="231.14" y2="297.18" width="0.1524" layer="91"/>
+<wire x1="238.76" y1="294.64" x2="231.14" y2="294.64" width="0.1524" layer="91"/>
 <pinref part="Q1" gate="G$1" pin="G"/>
 </segment>
