File: eagle/system-controller.brd (EAGLE design)
At the start: 99 x 100 mm, 220 parts, among them IC1 TS4100, Q1 MOSFET-P-N-PAIR, Q10 MOSFET-P-N-PAIR, Q11 MOSFET-P-N-PAIR, Q12 MOSFET-P-N-PAIR, Q13 MOSFET-P-N-PAIR, Q14 MOSFET-P-N-PAIR, Q15 MOSFET-P-N-PAIR, Q16 MOSFET-P-N-PAIR, Q17 MOSFET-P-N-PAIR, Q18 MOSFET-P-N-PAIR, Q19 MOSFET-P-N-PAIR, Q2 MOSFET-P-N-PAIR, Q3 DNP/NTR4101P, Q4 DNP/NTR4101P, Q5 DNP/NTR4101P, Q6 DNP/NTR4101P, Q7 MOSFET-P-N-PAIR, Q8 MOSFET-P-N-PAIR, Q9 MOSFET-P-N-PAIR, SW1 TPS25944LRVCRWQFN-20-3X4, SW2 TPS25944LRVCRWQFN-20-3X4, SW3 TPS25944LRVCRWQFN-20-3X4, SW4 TPS25944LRVCRWQFN-20-3X4, SW5 TPS25944LRVCRWQFN-20-3X4, SW6 TPS25944LRVCRWQFN-20-3X4, SW7 TPS25944LRVCRWQFN-20-3X4, SW8 TPS25944LRVCRWQFN-20-3X4, U1 MEGA128-A, X1 CRYSTAL-ABRACON-ABM3-SMD

Commit message: Fixed nuclear option. Fixed ERCs. Found ERCs in ATMEGAS128, so broke that out of the default ATMEL library from CADSOFT and made our own (now in the oresat-eagle-libraries repo). Replaced test points with decent test point that wasn't 6,000 km wide, and had a better symbol. Fixed AREF, which shouldn't have been pulled high. Some OCD cleanup. ERCs now manageable.
Parts:
- removed TP27: TPSPAD1-13, testpad:P1-13
- added TP43, TP44, TP45: TEST-POINT, Tova:2MM-TEST-POINT
- TP10, TP11, TP12, TP13, TP14, TP15, TP16, TP17, TP18, TP19, TP2, TP20, TP21, TP22, TP23, TP24, TP25, TP26, TP28, TP29, TP3, TP30, TP31, TP32, TP33, TP34, TP35, TP36, TP37, TP38, TP39, TP4, TP40, TP41, TP42, TP5, TP6, TP7, TP8, TP9: value TPSPAD1-13 -> TEST-POINT; device testpad:P1-13 -> Tova:2MM-TEST-POINT
- U1: device atmel:TQFP64 -> atmegas128:TQFP64
- X1: value CRYSTAL-ABRACON-ABM3-SMD -> 8 MHz CRYSTAL-ABRACON-ABM3-SMD
- moved Q20 161.2 mm to (123.2, -14.0), turned to 90 degrees
- moved R67 153.2 mm to (117.4, -14.7), turned to 90 degrees
- moved R66 147.6 mm to (113.4, -14.7), turned to 90 degrees
- moved C31 142.1 mm to (109.4, -14.7), turned to 90 degrees
- moved D3 131.6 mm to (102.4, -12.0)
- moved R65 124.0 mm to (96.4, -14.7), turned to 90 degrees
- moved R64 118.5 mm to (92.4, -14.7), turned to 90 degrees
- moved R52 112.9 mm to (88.4, -14.7), turned to 90 degrees
- moved RUVLO8 107.4 mm to (84.4, -14.7), turned to 90 degrees
- moved TP5 102.6 mm to (10.6, -6.20), turned to 90 degrees
- moved RUVLO7 101.9 mm to (80.4, -14.7), turned to 90 degrees
- moved TP30 97.8 mm to (21.7, -6.20), turned to 90 degrees
- moved RUVLO6 96.5 mm to (76.4, -14.7), turned to 90 degrees
- moved TP28 95.9 mm to (14.3, -6.20)
- moved TP29 94.9 mm to (18.0, -6.20)
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Connections:
- net FC_UART_RX renamed UART_FC_RX
- net FC_UART_TX renamed UART_FC_TX
- net FC_UART_VCC renamed UART_FC_VCC
- net LGR_UART_RX renamed UART_LGR_RX
- net LGR_UART_TX renamed UART_LGR_TX
- net LGR_UART_VCC renamed UART_LGR_VCC
- net SCL renamed I2C-SCL
- net SDA renamed I2C-SDA
- removed net NUKEPIN: CF1.P$15, CF1.P$16, Q20.2
- new net N$104: U1.32
- new net NUCLEAROPTION_OUT: CF1.P$15, CF1.P$16, Q20.3, TP44.1
- net 3V: now also J1.2, R50.1, R57.1, R58.1, R59.1; no longer C27.2, U1.62
- net GND: now also Q20.2, R13.2, TP28.1, TP30.1, TP32.1, TP34.1, TP36.1, TP38.1, TP40.1, TP42.1; no longer TP28.TP, TP31.TP, TP33.TP, TP35.TP, TP37.TP, TP39.TP, TP41.TP, TP5.TP
- net N$101: now also TP39.1; no longer TP42.TP
- net N$109: now also TP43.1
- net N$11: now also J1.10
- net N$12: now also J1.6
- net N$13: now also J1.8
- net N$14: now also J1.4
- net N$24: no longer Q5.1
- net N$25: now also TP5.1; no longer TP29.TP
- net N$32: now also TP29.1; no longer TP30.TP
- net N$33: now also TP4.1; no longer TP4.TP
- net N$36: now also C27.2, U1.62; no longer C23.2, R12.1, U$8.1
- net N$59: now also TP31.1; no longer TP32.TP
- net N$69: now also TP41.1; no longer TP34.TP
- net N$77: now also TP37.1; no longer TP36.TP
- net N$85: now also TP35.1; no longer TP38.TP
- net N$93: now also TP33.1; no longer TP40.TP
- net PB0: now also TP7.1; no longer TP19.TP
- net PB1: now also TP8.1; no longer TP18.TP
- net PB2: now also TP9.1; no longer TP17.TP
- net PB3: now also TP15.1; no longer TP16.TP
- net PB4: now also TP16.1; no longer TP15.TP
- net PB5: now also TP17.1; no longer TP9.TP
- net PB6: now also TP18.1; no longer TP8.TP
- net PB7: now also TP19.1; no longer TP7.TP
- net PCB3_EN: now also TP11.1; no longer TP13.TP
- net RXD1: now also Q5.1
- net V+: now also C23.2, R12.1, U$8.1
- net VBUS: now also C15.2; no longer Q20.3
- net VCB0_!FLT: now also R50.2, TP26.1; no longer R59.1, R62.2, TP20.TP
- net VCB0_EN: now also TP14.1; no longer TP10.TP
- net VCB1_!FLT: now also R17.2, TP25.1; no longer R11.2, R58.1, TP21.TP
- net VCB1_EN: now also TP13.1; no longer TP11.TP
- net VCB2_!FLT: now also R57.2, TP24.1; no longer R17.2, R57.1, TP22.TP
- net VCB2_EN: now also TP12.1; no longer TP12.TP
- net VCB3_!FLT: now also R11.2, TP23.1; no longer R50.1, R60.2, TP23.TP
- net VCB4_!FLT: now also R58.2, TP22.1; no longer R59.2, TP24.TP
- net VCB4_EN: now also TP10.1; no longer TP14.TP
- net VCB5_!FLT: now also R62.2, TP21.1; no longer R58.2, TP25.TP
- net VCB5_EN: now also TP6.1; no longer TP2.TP
- net VCB6_!FLT: now also R59.2, TP20.1; no longer R57.2, TP26.TP
- net VCB6_EN: now also TP3.1; no longer TP3.TP
- net VCB7_!FLT: now also R60.2, TP45.1; no longer R50.2, TP27.TP
- net VCB7_EN: now also TP2.1; no longer TP6.TP
