File: eagle/system-controller.sch (EAGLE design)
At the start: 219 parts, among them IC1 TS4100, Q1 MOSFET-P-N-PAIR, Q10 MOSFET-P-N-PAIR, Q11 MOSFET-P-N-PAIR, Q12 MOSFET-P-N-PAIR, Q13 MOSFET-P-N-PAIR, Q14 MOSFET-P-N-PAIR, Q15 MOSFET-P-N-PAIR, Q16 MOSFET-P-N-PAIR, Q17 MOSFET-P-N-PAIR, Q18 MOSFET-P-N-PAIR, Q19 MOSFET-P-N-PAIR, Q2 MOSFET-P-N-PAIR, Q3 DNP/NTR4101P, Q4 DNP/NTR4101P, Q5 DNP/NTR4101P, Q6 DNP/NTR4101P, Q7 MOSFET-P-N-PAIR, Q8 MOSFET-P-N-PAIR, Q9 MOSFET-P-N-PAIR, SW1 TPS25944LRVCRWQFN-20-3X4, SW2 TPS25944LRVCRWQFN-20-3X4, SW3 TPS25944LRVCRWQFN-20-3X4, SW4 TPS25944LRVCRWQFN-20-3X4, SW5 TPS25944LRVCRWQFN-20-3X4, SW6 TPS25944LRVCRWQFN-20-3X4, SW7 TPS25944LRVCRWQFN-20-3X4, SW8 TPS25944LRVCRWQFN-20-3X4, U1 MEGA128-A, X1 CRYSTAL-ABRACON-ABM3-SMD

Commit message: Fixed nuclear option. Fixed ERCs. Found ERCs in ATMEGAS128, so broke that out of the default ATMEL library from CADSOFT and made our own (now in the oresat-eagle-libraries repo). Replaced test points with decent test point that wasn't 6,000 km wide, and had a better symbol. Fixed AREF, which shouldn't have been pulled high. Some OCD cleanup. ERCs now manageable.
Parts:
- removed TP27: TPSPAD1-13, testpad:TPSPAD1-13
- added TP43, TP44, TP45: TEST-POINT, Tova:TEST-POINT
- TP10, TP11, TP12, TP13, TP14, TP15, TP16, TP17, TP18, TP19, TP2, TP20, TP21, TP22, TP23, TP24, TP25, TP26, TP28, TP29, TP3, TP30, TP31, TP32, TP33, TP34, TP35, TP36, TP37, TP38, TP39, TP4, TP40, TP41, TP42, TP5, TP6, TP7, TP8, TP9: value TPSPAD1-13 -> TEST-POINT; device testpad:TPSPAD1-13 -> Tova:TEST-POINT
- U1: device atmel:MEGA128-A -> atmegas128:MEGA128-A
- X1: value CRYSTAL-ABRACON-ABM3-SMD -> 8 MHz CRYSTAL-ABRACON-ABM3-SMD
Connections:
- net FC_UART_RX renamed UART_FC_RX
- net FC_UART_TX renamed UART_FC_TX
- net FC_UART_VCC renamed UART_FC_VCC
- net LGR_UART_RX renamed UART_LGR_RX
- net LGR_UART_TX renamed UART_LGR_TX
- net LGR_UART_VCC renamed UART_LGR_VCC
- net SCL renamed I2C-SCL
- net SDA renamed I2C-SDA
- removed net NUKEPIN: CF1.15, CF1.16, Q20.S
- new net N$104: U1.(T2)PD7
- new net NUCLEAROPTION_OUT: CF1.15, CF1.16, Q20.D, TP44.1
- net 3V: now also J1.TMS, R50.1, R57.1, R58.1, R59.1; no longer C27.2, U1.AREF
- net GND: now also Q20.S, R13.2, TP28.1, TP30.1, TP32.1, TP34.1, TP36.1, TP38.1, TP40.1, TP42.1; no longer TP28.PP, TP31.PP, TP33.PP, TP35.PP, TP37.PP, TP39.PP, TP41.PP, TP5.PP
- net N$101: now also TP39.1; no longer TP42.PP
- net N$109: now also TP43.1
- net N$11: now also J1.SRST
- net N$12: now also J1.TDO
- net N$13: now also J1.TDI
- net N$14: now also J1.TCK
- net N$24: no longer Q5.G
- net N$25: now also TP5.1; no longer TP29.PP
- net N$32: now also TP29.1; no longer TP30.PP
- net N$33: now also TP4.1; no longer TP4.PP
- net N$36: now also C27.2, U1.AREF; no longer C23.2, R12.1, U$8.VIN
- net N$59: now also TP31.1; no longer TP32.PP
- net N$69: now also TP41.1; no longer TP34.PP
- net N$77: now also TP37.1; no longer TP36.PP
- net N$85: now also TP35.1; no longer TP38.PP
- net N$93: now also TP33.1; no longer TP40.PP
- net PB0: now also TP7.1; no longer TP19.PP
- net PB1: now also TP8.1; no longer TP18.PP
- net PB2: now also TP9.1; no longer TP17.PP
- net PB3: now also TP15.1; no longer TP16.PP
- net PB4: now also TP16.1; no longer TP15.PP
- net PB5: now also TP17.1; no longer TP9.PP
- net PB6: now also TP18.1; no longer TP8.PP
- net PB7: now also TP19.1; no longer TP7.PP
- net PCB3_EN: now also TP11.1; no longer TP13.PP
- net RXD1: now also Q5.G
- net V+: now also C23.2, R12.1, U$8.VIN
- net VBUS: now also C15.2; no longer Q20.D
- net VCB0_!FLT: now also R50.2, TP26.1; no longer R59.1, R62.2, TP20.PP
- net VCB0_EN: now also TP14.1; no longer TP10.PP
- net VCB1_!FLT: now also R17.2, TP25.1; no longer R11.2, R58.1, TP21.PP
- net VCB1_EN: now also TP13.1; no longer TP11.PP
- net VCB2_!FLT: now also R57.2, TP24.1; no longer R17.2, R57.1, TP22.PP
- net VCB2_EN: now also TP12.1; no longer TP12.PP
- net VCB3_!FLT: now also R11.2, TP23.1; no longer R50.1, R60.2, TP23.PP
- net VCB4_!FLT: now also R58.2, TP22.1; no longer R59.2, TP24.PP
- net VCB4_EN: now also TP10.1; no longer TP14.PP
- net VCB5_!FLT: now also R62.2, TP21.1; no longer R58.2, TP25.PP
- net VCB5_EN: now also TP6.1; no longer TP2.PP
- net VCB6_!FLT: now also R59.2, TP20.1; no longer R57.2, TP26.PP
- net VCB6_EN: now also TP3.1; no longer TP3.PP
- net VCB7_!FLT: now also R60.2, TP45.1; no longer R50.2, TP27.PP
- net VCB7_EN: now also TP2.1; no longer TP6.PP
Other:
- note added: ""Nuclear Option" system-wide hard shutdown"
- note added: "8 MHz"
- note added: "RH"
- note removed: "Hardware WatchDog"
- moved on the sheet: C1, C2, C23, C25, C26, C27, C28, C30, C31, C4, C40, C5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
