File: eagle/system-controller.sch (EAGLE design)
At the start: 224 parts, among them J1 1, Q1 MOSFET-P-N-PAIR, Q10 MOSFET-P-N-PAIR, Q11 DNP/NTR4101P, Q2 MOSFET-P-N-PAIR, Q3 DON3035L, Q4 MOSFET-P-N-PAIR, Q5 MOSFET-P-N-PAIR, Q6 MOSFET-P-N-PAIR, Q7 MOSFET-P-N-PAIR, Q8 MOSFET-P-N-PAIR, Q9 DNP/NTR4101P, U1 TPS25944LRVCRWQFN-20-3X4, U10 TPS25944LRVCRWQFN-20-3X4, U11 ACPL-M61L, U12 ACPL-M61L, U13 TPS25944LRVCRWQFN-20-3X4, U14 ACPL-M61L, U15 ACPL-M61L, U2 LP5907MFX-3.0, U3 TPS25944LRVCRWQFN-20-3X4, U4 TPS25944LRVCRWQFN-20-3X4, U5 TPS25944LRVCRWQFN-20-3X4, U6 TPS25944LRVCRWQFN-20-3X4, U7 ATMEGA128L-8A(U/N), U8 TS4100, U9 TPS25944LRVCRWQFN-20-3X4, X1 8 MHz CRYSTAL-ABRACON-ABM3-SMD

Commit message: Added 3V LED for power. Fixed a DRC error which wasn't caught earlier? How'd that happen? Also pushing gerbers, since some folks don't have EAGLE.
Parts:
- added LED13: DNP/GRN, psas_c3_team05:LED-0603
- added R76: DNP/1k, rcl_custom:R-US_0603-B-NOSILK
Connections:
- new net N$6: LED13.A, R76.2
- net 3V: now also R76.1
- net GND: now also LED13.K
Other:
- note added: "1.1"
Changed lines of the file:
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@@
 <attribute name="MPN" value="4-1676481-5"/>
 </part>
+<part name="R76" library="rcl_custom" deviceset="R-US_" device="0603-B-NOSILK" value="DNP/1k">
+<attribute name="DIST" value="digikey"/>
+<attribute name="DPN" value="1276-3484-1-ND"/>
+<attribute name="MFN" value="Samsung"/>
+<attribute name="MPN" value="RC1608F102CS"/>
+</part>
+<part name="LED13" library="psas_c3_team05" deviceset="LED" device="-0603" value="DNP/GRN">
+<attribute name="DIST" value="digikey"/>
+<attribute name="DPN" value="732-4971-1-ND"/>
+<attribute name="MFN" value="Wurth Electronics INC."/>
+<attribute name="MPN" value="150060GS75000"/>
+</part>
+<part name="GND2" library="psas_c3_team05" deviceset="GND" device=""/>
+<part name="3V-11" library="supply-3v" deviceset="3V" device=""/>
 </parts>
 <sheets>
@@
 <plain>
 <text x="455.93" y="30.48" size="2.54" layer="97">William Harrington, James Heath, Shan Quinney</text>
-<wire x1="129.54" y1="406.4" x2="205.74" y2="406.4" width="0.1524" layer="97" style="longdash"/>
-<wire x1="205.74" y1="406.4" x2="205.74" y2="360.68" width="0.1524" layer="97" style="longdash"/>
-<wire x1="205.74" y1="360.68" x2="129.54" y2="360.68" width="0.1524" layer="97" style="longdash"/>
+<wire x1="129.54" y1="406.4" x2="233.68" y2="406.4" width="0.1524" layer="97" style="longdash"/>
+<wire x1="233.68" y1="406.4" x2="233.68" y2="360.68" width="0.1524" layer="97" style="longdash"/>
+<wire x1="233.68" y1="360.68" x2="129.54" y2="360.68" width="0.1524" layer="97" style="longdash"/>
 <wire x1="129.54" y1="360.68" x2="129.54" y2="406.4" width="0.1524" layer="97" style="longdash"/>
 <text x="132.08" y="403.86" size="1.778" layer="97">LDO for System Controller (RH)
@@
 When all three pins are high the voltage at TP43 is 0.75V</text>
 <text x="307.34" y="345.44" size="1.778" layer="97">Look for TPs connected to GND!!!!!!</text>
+<text x="546.1" y="7.62" size="2.54" layer="97">1.1</text>
 </plain>
 <instances>
@@
 <attribute name="MPN" x="111.76" y="309.88" size="1.778" layer="96" rot="R270" display="off"/>
 </instance>
+<instance part="R76" gate="R" x="210.82" y="386.08" smashed="yes" rot="R270">
+<attribute name="NAME" x="213.36" y="386.08" size="1.778" layer="95"/>
+<attribute name="VALUE" x="213.36" y="383.54" size="1.778" layer="96"/>
+<attribute name="DIST" x="210.82" y="386.08" size="1.778" layer="96" rot="R270" display="off"/>
+<attribute name="DPN" x="210.82" y="386.08" size="1.778" layer="96" rot="R270" display="off"/>
+<attribute name="MFN" x="210.82" y="386.08" size="1.778" layer="96" rot="R270" display="off"/>
+<attribute name="MPN" x="210.82" y="386.08" size="1.778" layer="96" rot="R270" display="off"/>
+</instance>
+<instance part="LED13" gate="LED" x="210.82" y="375.92" smashed="yes">
+<attribute name="NAME" x="213.36" y="377.19" size="1.778" layer="95"/>
+<attribute name="VALUE" x="213.36" y="374.65" size="1.778" layer="96"/>
+<attribute name="DIST" x="210.82" y="375.92" size="1.778" layer="96" display="off"/>
+<attribute name="DPN" x="210.82" y="375.92" size="1.778" layer="96" display="off"/>
+<attribute name="MPN" x="210.82" y="375.92" size="1.778" layer="96" display="off"/>
+<attribute name="MFN" x="210.82" y="375.92" size="1.778" layer="96" display="off"/>
+</instance>
+<instance part="GND2" gate="1" x="210.82" y="370.84"/>
+<instance part="3V-11" gate="G$1" x="210.82" y="393.7"/>
 </instances>
 <busses>
@@
 <wire x1="228.6" y1="68.58" x2="228.6" y2="66.04" width="0.1524" layer="91"/>
 </segment>
+<segment>
+<pinref part="R76" gate="R" pin="1"/>
+<pinref part="3V-11" gate="G$1" pin="3V"/>
+</segment>
 </net>
 <net name="N$26" class="0">
@@
 <pinref part="U13" gate="G$1" pin="PGHT"/>
 </segment>
+<segment>
+<pinref part="LED13" gate="LED" pin="K"/>
+<pinref part="GND2" gate="1" pin="GND"/>
+</segment>
 </net>
 <net name="N$50" class="0">
@@
 </segment>
 </net>
+<net name="N$6" class="0">
+<segment>
+<pinref part="R76" gate="R" pin="2"/>
+<pinref part="LED13" gate="LED" pin="A"/>
+</segment>
+</net>
